Commit message: solve bug in mapping package and turing,add a probability-grid-mapping ,some bugs and next version will solve them and add some features

File: wangbx_robot_description/urdf/wangbx_robot.urdf.xacro (robot description, xacro)
@@ -20,5 +20,5 @@
       <collision name="base">
         <geometry>
-          <cylinder length="0.10938" radius="0.178"/>
+          <cylinder length="0.10" radius="0.1"/>
         </geometry>
         <origin xyz="0.0 0 0.05949" rpy="0 0 0"/>
